File: PHASE D/PCB Design/GPS_TRACKER/GPS_TRACKER.kicad_pcb (KiCad board)
At the start: 2 copper layers, 8 parts

Commit message: 1
Parts:
- moved BuckConverter1 67.5 mm to (159.3, 58.4)
- moved SMS1 67.5 mm to (142.2, 74.9)
- moved BuckConverter1 67.5 mm to (143.8, 58.3)
- moved GPS1 67.5 mm to (144.8, 110.5)
- moved SMS1 67.5 mm to (165.1, 77.5)
- moved STM32F4_Discovery_Header 67.5 mm to (152.4, 88.9)
- moved BuckConverter1 67.5 mm to (159.5, 49.1)
- moved BuckConverter1 67.5 mm to (144.1, 49.2)
Other:
- board outline added: 73.7 x 104.1 mm
