File: PHASE D/PCB Design/GPS_TRACKER/GPS_TRACKER.kicad_sch (KiCad schematic)
At the start: 3 parts

Commit message: 1
Other:
- note added: "~ This are the componets of the project and are place onto a sheild for the STM32 Discovery Board ~ See PCB layout and gerber files to see how etherything will be wired for the sheild"
- company: (none) -> University of Denver 
- title: (none) -> STM32 GPS Shield 
- moved on the sheet: BuckConverter1, GPS1, SMS1
